File: eagle/Pinball10/Pinball10.brd (EAGLE design)
At the start: 63.5 x 40.6 mm, 49 parts, among them J1 UB-M5BR-DM14, Q1 MOSFET-NCHANNEL2N7002PW, U1 CYBLE-014008-00, U2 MMA8452Q, U3 PCA9306, U4 V_REG_317SMD

Commit message: labeling done
Parts:
- GND: value PTR1PAD1-13 -> GND
- renumbered JP1 to M0+, JP2 to M1+, LEDBANK0 to BANK0, TP1 to V50, TP2 to GND, TP3 to V33
Connections:
- removed net VDD: LCD.2
- net V50: now also LCD.2
Routing:
- net V50: track 131.6 -> 134.9 mm
- net GND: track 7.79 -> 5.45 mm, vias 98 -> 92
Other:
- board text added: "+"
- board text added: "-"
- board text added: "0 0"
- board text added: "0 1"
- board text added: "0 2"
- board text added: "0 3"
- board text added: "1 0"
- board text added: "1 1"
- board text added: "1 2"
- board text added: "1 3"
- board text added: "2 0"
- board text added: "2 1"
- board text added: "2 2"
- board text added: "2 3"
- board text added: "3 0"
- board text added: "3 1"
- board text added: "3 2"
- board text added: "3 3"
- board text added: "5V"
- board text added: "BUZZER 0"
- board text added: "BUZZER 1"
- board text added: "GND"
- board text added: "Newton's Attic"
- board text added: "Pinball Wizard 1.0"
- board text added: "ROW COL"
- board text added: "SCLK"
- board text added: "SDAT"
- board text added: "iotexpert.com"
- board text added: "www.iotexpert.com"

Commit message: maybe 1.0 board?
Parts:
- M0+, M1+: value M02PTH -> m
Routing:
- net GND: vias 92 -> 91

Commit message: fixed errors from ERC (and found a real layout error
Connections:
- removed net N$29: U2.10
- removed net N$9: U2.9
- net GND: now also U2.10
Routing:
- net GND: track 5.45 -> 7.47 mm
Changed lines of the file:
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@@
 <wire x1="14.994" y1="24.897" x2="14.986" y2="24.897" width="0.254" layer="1"/>
 <wire x1="14.986" y1="24.897" x2="14.986" y2="25.908" width="0.254" layer="1"/>
+<contactref element="U2" pad="10"/>
+<wire x1="15.994" y1="24.897" x2="15.9258" y2="24.897" width="0.254" layer="1"/>
+<wire x1="15.9258" y1="24.897" x2="15.9258" y2="25.908" width="0.254" layer="1"/>
+<wire x1="15.9258" y1="25.908" x2="14.986" y2="25.908" width="0.254" layer="1"/>
 </signal>
 <signal name="M1R">
@@
 <via x="14.097" y="20.1168" extent="1-16" drill="0.3302"/>
 </signal>
-<signal name="N$9">
-<contactref element="U2" pad="9"/>
-</signal>
 <signal name="SDA33">
 <contactref element="U2" pad="6"/>
@@
 <wire x1="15.0114" y1="21.0312" x2="14.986" y2="20.966" width="0.1524" layer="1"/>
 </signal>
-<signal name="N$29">
-<contactref element="U2" pad="10"/>
-</signal>
 <signal name="V33" class="1">

Commit message: final 1.0c board
Parts:
- renumbered SG2 to 1
Other:
- board text added: "SWDIO"
- board text added: "V50"
- board text added: "XRES"

Commit message: added some values to the schematic as I filled in the BOM
Parts:
- C1: value (none) -> 0.1uF
- C2: value (none) -> 1uF
- R1, R2, R3, R4: value (none) -> 330
- R10, R9: value (none) -> 560
- R12, R13: value (none) -> 2.2K
- R5: value (none) -> 1.8K
- R6: value (none) -> 1.2K
Changed lines of the file:
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@@
 <layer number="19" name="Unrouted" color="6" fill="1" visible="no" active="yes"/>
 <layer number="20" name="Dimension" color="15" fill="1" visible="yes" active="yes"/>
-<layer number="21" name="tPlace" color="7" fill="1" visible="no" active="yes"/>
-<layer number="22" name="bPlace" color="7" fill="1" visible="no" active="yes"/>
+<layer number="21" name="tPlace" color="7" fill="1" visible="yes" active="yes"/>
+<layer number="22" name="bPlace" color="7" fill="1" visible="yes" active="yes"/>
 <layer number="23" name="tOrigins" color="15" fill="1" visible="no" active="yes"/>
 <layer number="24" name="bOrigins" color="15" fill="1" visible="no" active="yes"/>
-<layer number="25" name="tNames" color="7" fill="1" visible="no" active="yes"/>
+<layer number="25" name="tNames" color="7" fill="1" visible="yes" active="yes"/>
 <layer number="26" name="bNames" color="7" fill="1" visible="yes" active="yes"/>
 <layer number="27" name="tValues" color="7" fill="1" visible="no" active="yes"/>
 <layer number="28" name="bValues" color="7" fill="1" visible="no" active="yes"/>
 <layer number="29" name="tStop" color="7" fill="3" visible="no" active="yes"/>
-<layer number="30" name="bStop" color="7" fill="6" visible="yes" active="yes"/>
+<layer number="30" name="bStop" color="7" fill="6" visible="no" active="yes"/>
 <layer number="31" name="tCream" color="7" fill="4" visible="no" active="yes"/>
-<layer number="32" name="bCream" color="7" fill="5" visible="yes" active="yes"/>
+<layer number="32" name="bCream" color="7" fill="5" visible="no" active="yes"/>
 <layer number="33" name="tFinish" color="6" fill="3" visible="no" active="yes"/>
 <layer number="34" name="bFinish" color="6" fill="6" visible="no" active="yes"/>
@@
 <attribute name="VALUE" x="38.5064" y="42.4688" size="1.27" layer="27" rot="R180"/>
 </element>
-<element name="R1" library="SparkFun" package="0805" value="" x="22.098" y="32.258" locked="yes" smashed="yes" rot="R270">
+<element name="R1" library="SparkFun" package="0805" value="330" x="22.098" y="32.258" locked="yes" smashed="yes" rot="R270">
 <attribute name="NAME" x="22.9235" y="33.02" size="0.762" layer="25" font="vector" ratio="18" rot="R270"/>
 <attribute name="VALUE" x="20.701" y="33.274" size="0.4064" layer="27" rot="R270"/>
 </element>
-<element name="R2" library="SparkFun" package="0805" value="" x="19.304" y="32.258" locked="yes" smashed="yes" rot="R270">
+<element name="R2" library="SparkFun" package="0805" value="330" x="19.304" y="32.258" locked="yes" smashed="yes" rot="R270">
 <attribute name="NAME" x="20.3835" y="32.766" size="0.762" layer="25" font="vector" ratio="18" rot="R270"/>
 <attribute name="VALUE" x="17.907" y="33.274" size="0.4064" layer="27" rot="R270"/>
 </element>
-<element name="R3" library="SparkFun" package="0805" value="" x="16.764" y="32.258" locked="yes" smashed="yes" rot="R270">
+<element name="R3" library="SparkFun" package="0805" value="330" x="16.764" y="32.258" locked="yes" smashed="yes" rot="R270">
 <attribute name="NAME" x="17.5895" y="33.02" size="0.762" layer="25" font="vector" ratio="18" rot="R270"/>
 <attribute name="VALUE" x="15.367" y="33.274" size="0.4064" layer="27" rot="R270"/>
 </element>
-<element name="R4" library="SparkFun" package="0805" value="" x="14.478" y="32.258" locked="yes" smashed="yes" rot="R270">
+<element name="R4" library="SparkFun" package="0805" value="330" x="14.478" y="32.258" locked="yes" smashed="yes" rot="R270">
 <attribute name="NAME" x="15.3035" y="33.02" size="0.762" layer="25" font="vector" ratio="18" rot="R270"/>
 <attribute name="VALUE" x="13.081" y="33.274" size="0.4064" layer="27" rot="R270"/>
@@
 <attribute name="PROD_ID" value="IC-10023" x="10.16" y="25.654" size="1.778" layer="27" display="off"/>
 </element>
-<element name="R5" library="SparkFun-Passives" package="0805" value="" x="2.794" y="13.716" locked="yes" smashed="yes" rot="R90">
+<element name="R5" library="SparkFun-Passives" package="0805" value="1.8K" x="2.794" y="13.716" locked="yes" smashed="yes" rot="R90">
 <attribute name="NAME" x="5.08" y="14.1605" size="0.762" layer="25" font="vector" ratio="18" rot="R180"/>
 <attribute name="VALUE" x="4.191" y="12.7" size="0.4064" layer="27" rot="R90"/>
 </element>
-<element name="R6" library="SparkFun-Passives" package="0805" value="" x="3.81" y="16.51" locked="yes" smashed="yes">
+<element name="R6" library="SparkFun-Passives" package="0805" value="1.2K" x="3.81" y="16.51" locked="yes" smashed="yes">
 <attribute name="NAME" x="2.2479" y="16.0782" size="0.762" layer="25" ratio="18" rot="R90"/>
 <attribute name="VALUE" x="2.794" y="15.113" size="0.4064" layer="27"/>
@@
 <attribute name="VALUE" x="4.2545" y="21.6535" size="0.4064" layer="27"/>
 </element>
-<element name="C1" library="SparkFun-Capacitors" package="0805" value="" x="9.906" y="17.272" locked="yes" smashed="yes" rot="R90">
+<element name="C1" library="SparkFun-Capacitors" package="0805" value="0.1uF" x="9.906" y="17.272" locked="yes" smashed="yes" rot="R90">
 <attribute name="NAME" x="11.0744" y="19.6215" size="0.762" layer="25" ratio="18" rot="R180"/>
 <attribute name="VALUE" x="11.303" y="16.256" size="0.4064" layer="27" rot="R90"/>
 </element>
-<element name="C2" library="SparkFun-Capacitors" package="0805" value="" x="7.366" y="16.51" locked="yes" smashed="yes" rot="R180">
+<element name="C2" library="SparkFun-Capacitors" package="0805" value="1uF" x="7.366" y="16.51" locked="yes" smashed="yes" rot="R180">
 <attribute name="NAME" x="8.128" y="15.6845" size="0.762" layer="25" font="vector" ratio="18" rot="R180"/>
 <attribute name="VALUE" x="8.382" y="17.907" size="0.4064" layer="27" rot="R180"/>
@@
 <attribute name="VALUE" x="14.097" y="25.4" size="0.4064" layer="27" rot="R90"/>
 </element>
-<element name="R9" library="SparkFun-Passives" package="0805" value="" x="34.417" y="11.557" locked="yes" smashed="yes">
+<element name="R9" library="SparkFun-Passives" package="0805" value="560" x="34.417" y="11.557" locked="yes" smashed="yes">
 <attribute name="NAME" x="34.925" y="12.3825" size="0.762" layer="25" font="vector" ratio="18"/>
 <attribute name="VALUE" x="33.401" y="10.16" size="0.4064" layer="27"/>
 </element>
-<element name="R10" library="SparkFun-Passives" package="0805" value="" x="34.798" y="8.89" locked="yes" smashed="yes" rot="R90">
+<element name="R10" library="SparkFun-Passives" package="0805" value="560" x="34.798" y="8.89" locked="yes" smashed="yes" rot="R90">
 <attribute name="NAME" x="33.9725" y="8.128" size="0.762" layer="25" font="vector" ratio="18" rot="R90"/>
 <attribute name="VALUE" x="36.195" y="7.874" size="0.4064" layer="27" rot="R90"/>
@@
 <attribute name="VALUE" x="49.784" y="4.699" size="1.27" layer="27" rot="R180"/>
 </element>
-<element name="R12" library="SparkFun-Passives" package="0805" value="" x="9.144" y="30.734" locked="yes" smashed="yes" rot="R90">
+<element name="R12" library="SparkFun-Passives" package="0805" value="2.2K" x="9.144" y="30.734" locked="yes" smashed="yes" rot="R90">
 <attribute name="NAME" x="9.9695" y="31.496" size="0.762" layer="25" font="vector" ratio="18" rot="R270"/>
 <attribute name="VALUE" x="10.541" y="29.718" size="0.4064" layer="27" rot="R90"/>
 </element>
-<element name="R13" library="SparkFun-Passives" package="0805" value="" x="11.43" y="30.734" locked="yes" smashed="yes" rot="R270">
+<element name="R13" library="SparkFun-Passives" package="0805" value="2.2K" x="11.43" y="30.734" locked="yes" smashed="yes" rot="R270">
 <attribute name="NAME" x="12.2809" y="31.9786" size="0.762" layer="25" font="vector" ratio="18" rot="R270"/>
 <attribute name="VALUE" x="10.033" y="31.75" size="0.4064" layer="27" rot="R270"/>

Commit message: the board ... but with the crash
Parts:
- M1+: value m -> M02PTH
- moved R9 16.3 mm to (49.3, 18.4)
- moved M0+ 14.0 mm to (34.1, 18.8), turned to 270 degrees
- moved R10 13.2 mm to (46.8, 14.5), turned to 270 degrees
- moved M1+ 12.9 mm to (34.1, 21.9), turned to 90 degrees
- moved V50 11.0 mm to (7.70, 25.1)
- moved JP3 10.8 mm to (37.7, 1.45), turned to 0 degrees
- moved C5 5.41 mm to (9.58, 22.0), turned to 180 degrees
- moved R11 4.74 mm to (16.7, 11.0)
- moved HBRIDGE 4.04 mm to (27.2, 21.7), turned to 90 degrees
- moved V33 3.72 mm to (6.20, 13.7)
- moved U3 3.36 mm to (13.5, 25.9), turned to 90 degrees
- moved U2 2.93 mm to (13.1, 21.9)
- moved C3 2.67 mm to (12.7, 18.6)
- moved C4 2.38 mm to (11.3, 18.6)
- moved C1 2.18 mm to (9.25, 15.2)
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Routing:
- net SWCOL2: track 57.5 -> 144.9 mm, vias 5 -> 4
- net SWCOL0: track 59.7 -> 109.8 mm, vias 4 -> 3
- net GND: track 7.12 -> 32.8 mm, vias 91 -> 94
- net SWDIO: track 20.2 -> 44.3 mm
- net N$3: track 24.4 -> 6.01 mm
- net SWDCLK: track 14.7 -> 31.6 mm, vias 2 -> 1
- net LEDCOL0: track 26.2 -> 42.9 mm, vias 4 -> 2
- net SWCOL1: track 77.7 -> 61.2 mm, vias 6 -> 5
- net V33: track 48.3 -> 32.5 mm, vias 2 -> 0
- net SWROW1: track 24.0 -> 38.5 mm, vias 1 -> 2
- net N$11: track 19.4 -> 5.58 mm
- net BUZZER1: track 26.9 -> 39.0 mm, vias 1 -> 2
- net LEDCOL3: track 39.4 -> 50.6 mm
- net V50: track 134.9 -> 124.1 mm, vias 3 -> 1
- net SDA50: track 69.3 -> 60.3 mm, vias 3 -> 5
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- added copper zone on layer 1, net V50
Other:
- board text added: "Pinball Wizard 1.1"
- board text removed: "Pinball Wizard 1.0"

Commit message: completed 1.1 of board
Parts:
- removed J1: UB-M5BR-DM14, con-usb:UB-M5BR-DM14
- added X1: MINI-USB-SHIELD-UX60-MB-5S8, con-hirose:UX60-MB-5S8
Connections:
- net GND: now also X1.5; no longer J1.5
- net V50: now also X1.1; no longer J1.1
Routing:
- net SWCOL2: track 144.9 -> 79.5 mm
- net LEDROW2: track 78.6 -> 63.2 mm, vias 0 -> 1
- net SWCOL0: track 109.8 -> 98.9 mm, vias 3 -> 2
- net ACCELINT: track 28.0 -> 24.4 mm, vias 0 -> 2
- net V50: track 124.1 -> 122.6 mm, vias 1 -> 2
- net GND: vias 94 -> 101
