File: eagle/Pinball10/Pinball10.brd (EAGLE design)
At the start: 74.4 x 42.2 mm, 46 parts, among them M0+ m, M1+ M02PTH, U1 CYBLE-014008-00, U2 MMA8452Q, U4 V_REG_317SMD, X1 MINI-USB-SHIELD-UX60-MB-5S8

Commit message: Released version 1.2 of board
Parts:
- added JMP1, JMP2, JMP3, JMP4: 0R-JUMPB, jump-0r-smd:B0R-JMP
Connections:
- removed net VDD: U$2.VDD
- new net D1: JMP3.2, U$2.SCL
- new net D2: JMP4.2, U$2.SDA
- new net P1: JMP1.2, U$2.GND
- new net P2: JMP2.2, U$2.VDD
- net GND: now also JMP1.1, JMP2.1; no longer U$2.GND
- net SCL: now also JMP3.1, JMP4.1; no longer U$2.SCL
- net SDA: now also JMP3.3, JMP4.3; no longer U$2.SDA
- net V33: now also JMP1.3, JMP2.3
Routing:
- net V33: track 115.3 -> 126.0 mm, vias 2 -> 4
- net D2: track 0.00 -> 10.7 mm
- net D1: track 0.00 -> 6.25 mm
- net P1: track 0.00 -> 6.00 mm
- net P2: track 0.00 -> 5.98 mm
- net SCL: track 106.1 -> 102.5 mm, vias 4 -> 3
- net GND: vias 106 -> 113
Other:
- board text added: "COL ROW"
- board text added: "Pinball Wizard 1.2"
- board text added: "SCL"
- board text added: "SDA"
- board text added: "SWD"
- board text added: "V33"
- board text added: "V5"
- board text removed: "5V"
- board text removed: "Pinball Wizard 1.1"
- board text removed: "SDAT"
