File: eagle/Pinball10/xxx.brd (EAGLE design)
At the start: 74.4 x 42.2 mm, 46 parts, among them M0+ m, M1+ M02PTH, U1 CYBLE-014008-00, U2 MMA8452Q, U4 V_REG_317SMD, X1 MINI-USB-SHIELD-UX60-MB-5S8

Commit message: New layout
Parts:
- moved B1 0.43 mm to (66.2, 7.52), turned to 90 degrees
Routing:
- net SCL: track 106.1 -> 0.00 mm, vias 4 -> 0
- net SDA: track 76.0 -> 0.00 mm, vias 4 -> 0
- net LEDROW2: track 72.5 -> 0.00 mm, vias 2 -> 0
- net LEDROW1: track 57.0 -> 0.00 mm
- net V33: track 115.3 -> 59.5 mm, vias 2 -> 0
- net XRES: track 52.9 -> 0.00 mm, vias 5 -> 0
- net LEDROW3: track 50.0 -> 0.00 mm, vias 2 -> 0
- net SWCOL1: track 50.0 -> 0.00 mm, vias 4 -> 0
- net LC1: track 49.2 -> 0.00 mm
- net GND: track 48.0 -> 0.00 mm, vias 106 -> 0
- net SWCOL2: track 47.2 -> 0.00 mm, vias 3 -> 0
- net LEDROW0: track 46.9 -> 0.00 mm
- net SWCOL0: track 46.5 -> 0.00 mm, vias 4 -> 0
- net LC2: track 42.3 -> 0.00 mm, vias 2 -> 0
- net LC3: track 41.7 -> 0.00 mm
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