File: eagle/Pinball10/Pinball10.sch (EAGLE design)
At the start: 46 parts, among them M0+ m, M1+ M02PTH, U1 CYBLE-014008-00, U2 MMA8452Q, U4 V_REG_317SMD, X1 MINI-USB-SHIELD-UX60-MB-5S8

Commit message: Released version 1.2 of board
Parts:
- added JMP1, JMP2, JMP3, JMP4: 0R-JUMPB, jump-0r-smd:0R-JUMPB
Connections:
- removed net VDD: U$2.VDD
- new net D1: JMP3-0R.2, U$2.SCL
- new net D2: JMP4-0R.2, U$2.SDA
- new net P1: JMP1-0R.2, U$2.GND
- new net P2: JMP2-0R.2, U$2.VDD
- net GND: now also JMP1-0R.1, JMP2-0R.1; no longer U$2.GND
- net SCL: now also JMP3-0R.1, JMP4-0R.1; no longer U$2.SCL
- net SDA: now also JMP3-0R.3, JMP4-0R.3; no longer U$2.SDA
- net V33: now also JMP1-0R.3, JMP2-0R.3
Changed lines of the file:
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@@
 <part name="JP1" library="SparkFun-Connectors" deviceset="M03" device="PTH"/>
 <part name="U$2" library="IOTExpert" deviceset="U8G-096-OLED" device=""/>
+<part name="JMP1" library="jump-0r-smd" deviceset="0R-JUMP" device="B"/>
+<part name="JMP2" library="jump-0r-smd" deviceset="0R-JUMP" device="B"/>
+<part name="JMP3" library="jump-0r-smd" deviceset="0R-JUMP" device="B"/>
+<part name="JMP4" library="jump-0r-smd" deviceset="0R-JUMP" device="B"/>
 </parts>
 <sheets>
@@
 <instance part="X1" gate="G$1" x="45.72" y="99.06"/>
 <instance part="U$2" gate="G$1" x="27.94" y="5.08"/>
+<instance part="JMP1" gate="-0R" x="-48.26" y="78.74"/>
+<instance part="JMP1" gate="G$2" x="-48.26" y="81.28"/>
+<instance part="JMP2" gate="-0R" x="-48.26" y="68.58"/>
+<instance part="JMP2" gate="G$2" x="-48.26" y="68.58"/>
+<instance part="JMP3" gate="-0R" x="-48.26" y="58.42"/>
+<instance part="JMP3" gate="G$2" x="-48.26" y="60.96"/>
+<instance part="JMP4" gate="-0R" x="-48.26" y="48.26"/>
+<instance part="JMP4" gate="G$2" x="-48.26" y="50.8"/>
 </instances>
 <busses>
@@
 </segment>
 <segment>
-<pinref part="U$2" gate="G$1" pin="GND"/>
-<wire x1="-5.08" y1="22.86" x2="-25.4" y2="22.86" width="0.1524" layer="91"/>
-<label x="-22.86" y="22.86" size="1.778" layer="95"/>
+<pinref part="JMP1" gate="-0R" pin="1"/>
+<wire x1="-48.26" y1="81.28" x2="-55.88" y2="81.28" width="0.1524" layer="91"/>
+<label x="-55.88" y="81.28" size="1.778" layer="95"/>
+</segment>
+<segment>
+<pinref part="JMP2" gate="-0R" pin="1"/>
+<wire x1="-48.26" y1="71.12" x2="-55.88" y2="71.12" width="0.1524" layer="91"/>
+<label x="-55.88" y="71.12" size="1.778" layer="95"/>
 </segment>
 </net>
@@
 <label x="116.84" y="76.2" size="1.778" layer="95"/>
 </segment>
+<segment>
+<pinref part="JMP1" gate="-0R" pin="3"/>
+<wire x1="-48.26" y1="76.2" x2="-55.88" y2="76.2" width="0.1524" layer="91"/>
+<label x="-55.88" y="76.2" size="1.778" layer="95"/>
+</segment>
+<segment>
+<pinref part="JMP2" gate="-0R" pin="3"/>
+<wire x1="-48.26" y1="66.04" x2="-55.88" y2="66.04" width="0.1524" layer="91"/>
+<label x="-55.88" y="66.04" size="1.778" layer="95"/>
+</segment>
 </net>
 <net name="SCL" class="0">
@@
 </segment>
 <segment>
+<pinref part="JMP3" gate="-0R" pin="1"/>
+<wire x1="-48.26" y1="60.96" x2="-55.88" y2="60.96" width="0.1524" layer="91"/>
+<label x="-55.88" y="60.96" size="1.778" layer="95"/>
+</segment>
+<segment>
+<pinref part="JMP4" gate="-0R" pin="1"/>
+<wire x1="-48.26" y1="50.8" x2="-55.88" y2="50.8" width="0.1524" layer="91"/>
+<label x="-55.88" y="50.8" size="1.778" layer="95"/>
+</segment>
+</net>
+<net name="SDA" class="0">
+<segment>
+<pinref part="U1" gate="U1" pin="P0.4/SDA0"/>
+<wire x1="20.32" y1="53.34" x2="10.16" y2="53.34" width="0.1524" layer="91"/>
+<label x="10.16" y="53.34" size="1.778" layer="95"/>
+</segment>
+<segment>
+<pinref part="R13" gate="G$1" pin="1"/>
+<wire x1="106.68" y1="76.2" x2="93.98" y2="76.2" width="0.1524" layer="91"/>
+<label x="93.98" y="76.2" size="1.778" layer="95"/>
+</segment>
+<segment>
+<pinref part="JMP3" gate="-0R" pin="3"/>
+<wire x1="-48.26" y1="55.88" x2="-55.88" y2="55.88" width="0.1524" layer="91"/>
+<label x="-55.88" y="55.88" size="1.778" layer="95"/>
+</segment>
+<segment>
+<pinref part="JMP4" gate="-0R" pin="3"/>
+<wire x1="-48.26" y1="45.72" x2="-55.88" y2="45.72" width="0.1524" layer="91"/>
+<label x="-55.88" y="45.72" size="1.778" layer="95"/>
+</segment>
+</net>
+<net name="ACCELINT" class="0">
+<segment>
+<pinref part="U1" gate="U1" pin="P3.2"/>
+<wire x1="55.88" y1="60.96" x2="63.5" y2="60.96" width="0.1524" layer="91"/>
+<label x="55.88" y="60.96" size="1.778" layer="95"/>
+</segment>
+</net>
+<net name="N$3" class="0">
+<segment>
+<pinref part="B0" gate="B1" pin="BUTTON"/>
+<wire x1="114.3" y1="30.48" x2="106.68" y2="30.48" width="0.1524" layer="91"/>
+<pinref part="R9" gate="G$1" pin="2"/>
+</segment>
+</net>
+<net name="N$11" class="0">
+<segment>
+<pinref part="B1" gate="B1" pin="BUTTON"/>
+<wire x1="114.3" y1="58.42" x2="109.22" y2="58.42" width="0.1524" layer="91"/>
+<pinref part="R10" gate="G$1" pin="2"/>
+</segment>
+</net>
+<net name="V50" class="1">
+<segment>
+<wire x1="40.64" y1="104.14" x2="25.4" y2="104.14" width="0.1524" layer="91"/>
+<label x="25.4" y="104.14" size="1.778" layer="95"/>
+<pinref part="X1" gate="G$1" pin="1"/>
+</segment>
+<segment>
+<wire x1="48.26" y1="7.62" x2="63.5" y2="7.62" width="0.1524" layer="91"/>
+<label x="50.8" y="7.62" size="1.778" layer="95"/>
+<pinref part="JP3" gate="G$1" pin="1"/>
+</segment>
+</net>
+<net name="P1" class="1">
+<segment>
+<pinref part="U$2" gate="G$1" pin="GND"/>
+<wire x1="-5.08" y1="22.86" x2="-25.4" y2="22.86" width="0.1524" layer="91"/>
+<label x="-22.86" y="22.86" size="1.778" layer="95"/>
+</segment>
+<segment>
+<pinref part="JMP1" gate="-0R" pin="2"/>
+<wire x1="-45.72" y1="78.74" x2="-33.02" y2="78.74" width="0.1524" layer="91"/>
+<label x="-43.18" y="78.74" size="1.778" layer="95"/>
+</segment>
+</net>
+<net name="P2" class="1">
+<segment>
+<pinref part="U$2" gate="G$1" pin="VDD"/>
+<wire x1="-5.08" y1="17.78" x2="-25.4" y2="17.78" width="0.1524" layer="91"/>
+<label x="-22.86" y="17.78" size="1.778" layer="95"/>
+</segment>
+<segment>
+<pinref part="JMP2" gate="-0R" pin="2"/>
+<wire x1="-45.72" y1="68.58" x2="-33.02" y2="68.58" width="0.1524" layer="91"/>
+<label x="-43.18" y="68.58" size="1.778" layer="95"/>
+</segment>
+</net>
+<net name="D1" class="0">
+<segment>
 <pinref part="U$2" gate="G$1" pin="SCL"/>
 <wire x1="-5.08" y1="12.7" x2="-25.4" y2="12.7" width="0.1524" layer="91"/>
 <label x="-22.86" y="12.7" size="1.778" layer="95"/>
 </segment>
-</net>
-<net name="SDA" class="0">
-<segment>
-<pinref part="U1" gate="U1" pin="P0.4/SDA0"/>
-<wire x1="20.32" y1="53.34" x2="10.16" y2="53.34" width="0.1524" layer="91"/>
-<label x="10.16" y="53.34" size="1.778" layer="95"/>
-</segment>
-<segment>
-<pinref part="R13" gate="G$1" pin="1"/>
-<wire x1="106.68" y1="76.2" x2="93.98" y2="76.2" width="0.1524" layer="91"/>
-<label x="93.98" y="76.2" size="1.778" layer="95"/>
-</segment>
+<segment>
+<pinref part="JMP3" gate="-0R" pin="2"/>
+<wire x1="-45.72" y1="58.42" x2="-33.02" y2="58.42" width="0.1524" layer="91"/>
+<label x="-43.18" y="58.42" size="1.778" layer="95"/>
+</segment>
+</net>
+<net name="D2" class="0">
 <segment>
 <pinref part="U$2" gate="G$1" pin="SDA"/>
@@
 <label x="-22.86" y="7.62" size="1.778" layer="95"/>
 </segment>
-</net>
-<net name="ACCELINT" class="0">
-<segment>
-<pinref part="U1" gate="U1" pin="P3.2"/>
-<wire x1="55.88" y1="60.96" x2="63.5" y2="60.96" width="0.1524" layer="91"/>
-<label x="55.88" y="60.96" size="1.778" layer="95"/>
-</segment>
-</net>
-<net name="N$3" class="0">
-<segment>
-<pinref part="B0" gate="B1" pin="BUTTON"/>
-<wire x1="114.3" y1="30.48" x2="106.68" y2="30.48" width="0.1524" layer="91"/>
-<pinref part="R9" gate="G$1" pin="2"/>
-</segment>
-</net>
-<net name="N$11" class="0">
-<segment>
-<pinref part="B1" gate="B1" pin="BUTTON"/>
-<wire x1="114.3" y1="58.42" x2="109.22" y2="58.42" width="0.1524" layer="91"/>
-<pinref part="R10" gate="G$1" pin="2"/>
-</segment>
-</net>
-<net name="V50" class="1">
-<segment>
-<wire x1="40.64" y1="104.14" x2="25.4" y2="104.14" width="0.1524" layer="91"/>
-<label x="25.4" y="104.14" size="1.778" layer="95"/>
-<pinref part="X1" gate="G$1" pin="1"/>
-</segment>
-<segment>
-<wire x1="48.26" y1="7.62" x2="63.5" y2="7.62" width="0.1524" layer="91"/>
-<label x="50.8" y="7.62" size="1.778" layer="95"/>
-<pinref part="JP3" gate="G$1" pin="1"/>
-</segment>
-</net>
-<net name="VDD" class="0">
-<segment>
-<pinref part="U$2" gate="G$1" pin="VDD"/>
-<wire x1="-5.08" y1="17.78" x2="-25.4" y2="17.78" width="0.1524" layer="91"/>
-<label x="-22.86" y="17.78" size="1.778" layer="95"/>
-</segment>
-</net>
+<segment>
+<pinref part="JMP4" gate="-0R" pin="2"/>
+<wire x1="-45.72" y1="48.26" x2="-33.02" y2="48.26" width="0.1524" layer="91"/>
+<label x="-43.18" y="48.26" size="1.778" layer="95"/>
+</segment>
+</net>
